File: boards/koov-shield3/koov-shield3.kicad_sch (KiCad schematic)
At the start: 24 parts, among them J1 Power, J2 Digital/PWM, J3 Analog, J4 Digital/PWM, SW1 SW_DPDT

Commit message: Support reverse-insertion-proof.
Parts:
- added UTL1: Conn_01x03, Connector_PinHeader_2.54mm:PinHeader_1x03_P2.54mm_Vertical, symbol Connector_Generic:Conn_01x03
Connections:
- net +3.3V: now also MD2.2 (Pin_2), UTL1.2 (Pin_2)
- net 11: now also UTL1.1 (Pin_1); no longer MD2.2 (Pin_2)
- net GND: now also UTL1.3 (Pin_3)

Commit message: Wiring UARTs to the unused connector.
Parts:
- added J5: RS1-02-G, CONN_RS1-02-G_ADM, symbol 2025-03-12_10-05-33:RS1-02-G
Connections:
- net 0: now also J5.1
- net 1: now also J5.2
Changed lines of the file:
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@@
 	(wire
 		(pts
+			(xy 259.08 68.58) (xy 262.89 68.58)
+		)
+		(stroke
+			(width 0)
+			(type default)
+		)
+	)
+	(wire
+		(pts
 			(xy 59.69 58.42) (xy 46.99 58.42)
 		)
@@
 	(wire
 		(pts
+			(xy 259.08 71.12) (xy 262.89 71.12)
+		)
+		(stroke
+			(width 0)
+			(type default)
+		)
+	)
+	(wire
+		(pts
 			(xy 34.29 99.06) (xy 34.29 109.22)
 		)
@@
 		)
 	)
+	(label "1"
+		(at 260.35 71.12 0)
+		(fields_autoplaced yes)
+		(effects
+			(font
+				(size 1.27 1.27)
+			)
+			(justify left bottom)
+		)
+	)
 	(label "*5"
 		(at 100.33 63.5 180)
@@
 		)
 	)
+	(label "0"
+		(at 260.35 68.58 0)
+		(fields_autoplaced yes)
+		(effects
+			(font
+				(size 1.27 1.27)
+			)
+			(justify left bottom)
+		)
+	)
 	(label "DC0_OUT0"
 		(at 190.5 120.65 0)
@@
 					(unit 1)
 				)
+			)
+		)
+	)
+	(symbol
+		(lib_id "2025-03-12_10-05-33:RS1-02-G")
+		(at 262.89 68.58 0)
+		(unit 1)
+		(exclude_from_sim no)
+		(in_bom yes)
+		(on_board yes)
+		(dnp no)
+		(property "Reference" "J5"
+			(at 270.256 62.992 0)
+			(effects
+				(font
+					(size 1.524 1.524)
+				)
+				(justify left)
+			)
+		)
+		(property "Value" "RS1-02-G"
+			(at 265.176 77.47 0)
+			(effects
+				(font
+					(size 1.524 1.524)
+				)
+				(justify left)
+			)
+		)
+		(property "Footprint" "CONN_RS1-02-G_ADM"
+			(at 262.89 68.58 0)
+			(effects
+				(font
+					(size 1.27 1.27)
+					(italic yes)
+				)
+				(hide yes)
+			)
+		)
+		(property "Datasheet" "RS1-02-G"
+			(at 262.89 68.58 0)
+			(effects
+				(font
+					(size 1.27 1.27)
+					(italic yes)
+				)
+				(hide yes)
+			)
+		)
+		(property "Description" ""
+			(at 262.89 68.58 0)
+			(effects
+				(font
+					(size 1.27 1.27)
+				)
+				(hide yes)
+			)
+		)
+		(pin "1"
+		)
+		(pin "2"
+		)
+		(instances
+			(project ""
+				(path "/e63e39d7-6ac0-4ffd-8aa3-1841a4541b55"
+					(reference "J5")
+					(unit 1)
+				)
